Commit message: Refactor ParkourEnv parameters and add debugging scripts
- Adjusted agent height and reward scales in ParkourEnv to improve balance and risk-taking behavior.
- Modified the reset method to ensure a fresh physics client is created for each episode.
- Introduced several debugging scripts:
  - `debug_fall.py`: Added debug information for fall detection.
  - `debug_spawn.py`: Isolated spawn position testing with and without LevelGenerator.
  - `debug_spawn2.py`: Tested self-collision handling.
  - `debug_spawn3.py`: Evaluated fixed base behavior and foot positions.
  - `debug_spawn4.py`: Verified behavior with self-collision disabled.
  - `debug_spawn5.py`: Checked contact points during simulation.
  - `debug_spawn6.py`: Tested agent spawning at a height of 1.4m.
- Added a quick test script `test_env.py` for initial environment validation.

File: assets/humanoid.urdf (robot description, URDF)
Before this commit: robot humanoid, 12 links, 11 joints
Links:
- link foot_L: geometry collision box size=0.26 0.10 0.05; visual box size=0.26 0.10 0.05
- link foot_R: geometry collision box size=0.26 0.10 0.05; visual box size=0.26 0.10 0.05
- link lower_arm_L: geometry collision cylinder length=0.22 radius=0.03; visual cylinder length=0.22 radius=0.03
- link lower_arm_R: geometry collision cylinder length=0.22 radius=0.03; visual cylinder length=0.22 radius=0.03
- link shin_L: geometry collision cylinder length=0.40 radius=0.05; visual cylinder length=0.40 radius=0.05
- link shin_R: geometry collision cylinder length=0.40 radius=0.05; visual cylinder length=0.40 radius=0.05
- link thigh_L: geometry collision cylinder length=0.40 radius=0.07; visual cylinder length=0.40 radius=0.07
- link thigh_R: geometry collision cylinder length=0.40 radius=0.07; visual cylinder length=0.40 radius=0.07
- link torso: geometry collision box size=0.18 0.28 0.65; visual box size=0.18 0.28 0.65
- link upper_arm_L: geometry collision cylinder length=0.24 radius=0.04; visual cylinder length=0.24 radius=0.04
- link upper_arm_R: geometry collision cylinder length=0.24 radius=0.04; visual cylinder length=0.24 radius=0.04
Joints:
- joint head_joint: origin xyz=0 0 0.32 rpy=0 0 0 -> xyz=0 0 0.45 rpy=0 0 0
- joint left_ankle: origin xyz=0 0 -0.36 rpy=0 0 0 -> xyz=0 0 -0.40 rpy=0 0 0
- joint left_elbow: origin xyz=0 0 -0.28 rpy=0 0 0 -> xyz=0 0 -0.24 rpy=0 0 0
- joint left_hip: origin xyz=0 0.09 -0.23 rpy=0 0 0 -> xyz=0 0.10 -0.30 rpy=0 0 0
- joint left_knee: origin xyz=0 0 -0.38 rpy=0 0 0 -> xyz=0 0 -0.40 rpy=0 0 0
- joint left_shoulder: origin xyz=0 0.17 0.17 rpy=0 0 0 -> xyz=0 0.19 0.25 rpy=0 0 0
- joint right_ankle: origin xyz=0 0 -0.36 rpy=0 0 0 -> xyz=0 0 -0.40 rpy=0 0 0
- joint right_elbow: origin xyz=0 0 -0.28 rpy=0 0 0 -> xyz=0 0 -0.24 rpy=0 0 0
- joint right_hip: origin xyz=0 -0.09 -0.23 rpy=0 0 0 -> xyz=0 -0.10 -0.30 rpy=0 0 0
- joint right_knee: origin xyz=0 0 -0.38 rpy=0 0 0 -> xyz=0 0 -0.40 rpy=0 0 0
- joint right_shoulder: origin xyz=0 -0.17 0.17 rpy=0 0 0 -> xyz=0 -0.19 0.25 rpy=0 0 0
